File: SmoothieBrainz_KiCad_V0.2/SmoothieBrainz - next round.sch (KiCad schematic (older format))
At the start: 127 parts, among them IC1 LPC1769, IC5 LD117ADT33TR, Q1 BSL207SP, Q2 12MHz, SW1 SW_TACT_4P_B, SW3 SW_TACT_4P_B, U2 HC_05, U3 USD-SOCKETUSD, X14 USBPTH

Commit message: Moved Items on to page Started to fix up components
Parts:
- Q2: symbol MICROBUILDER_CRYSTALTHIN -> MICROBUILDER_CRYSTAL
Connections:
- net labels added: +3.3V
Other:
- moved on the sheet: EXP1A, EXP1B, EXP1C, EXP1D, EXP1E, EXP1F, EXP1G, EXP1H, EXP1I, EXP1J, EXP2A, EXP2B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

Commit message: Fixed Inductors and Caps and 3.3V and GND
Parts:
- C1, C17, C18, C19, C20, C21, C22, C23, C24, C25, C28, C44, C64, C65, C67, C7: symbol RESISTOR_C-EUC0603 -> RCL_C-EU
- C10, C11, C12, C13, C14, C2, C3, C4, C5, C6, C8, C9: symbol RCL_C-EUC0603 -> RCL_C-EU
- L1: symbol SPARKFUN_INDUCTOR0603 -> SPARKFUN-PASSIVES_INDUCTOR
- L2: symbol SPARKFUN-PASSIVES_INDUCTORPWR -> SPARKFUN-PASSIVES_INDUCTOR

Commit message: Fixed up more components The remaining components will be deleted soon
Parts:
- C15, C16: value (none) -> ~; symbol RCL_CPOL-EUE2.5-7 -> RCL_CPOL-EU
- C26, C27: symbol RCL_CPOL-EUE2.5-7 -> RCL_CPOL-EU
- JP1: value (none) -> JP1; symbol PINHEAD_PINHD-2X7_90 -> PINHEAD_PINHD-2X7
- L1: value (none) -> ~
- LED1, LED2, LED3, LED4, LED5, LED9: value (none) -> ~; symbol LED_LEDCHIP-LED0805 -> LED_LED
- R1, R10, R11, R12, R13, R14, R15, R17, R18, R2, R3, R51, R7, R77, R8, R9: symbol RESISTOR_R-US_R0603 -> RESISTOR_R-US_
- RN1: symbol RESISTOR-DIL_4R-N0603-ARV -> RESISTOR-DIL_4R-N
- S1: value (none) -> sw1; symbol SPARKFUN_TAC_SWITCHSMD -> SPARKFUN_TAC_SWITCH
- S2: value (none) -> sw2; symbol SPARKFUN_TAC_SWITCHSMD -> SPARKFUN_TAC_SWITCH
- U3: symbol SPARKFUN-CONNECTORS_PETERMICROSDEBAY_USD-SOCKETUSD -> SPARKFUN-CONNECTORS_PETERMICROSDEBAY_USD-SOCKET
- X14: symbol SPARKFUN_USBPTH -> SPARKFUN_USB

Commit message: More Clean up of Sch
Parts:
- removed unit 0 of RN1 (x2)
- added unit 2 of RN1
- added unit 3 of RN1
- D1, D3: symbol MICROBUILDER_DIODESMA -> MICROBUILDER_DIODE
- D10, D11, D12, D7, D8, D9: symbol SEMICON-SMD-IPC_D-SOD-87 -> DP_DEVICES_DIODE
- D2: value (none) -> 214AC; symbol DP_DEVICES_DIODE-DO-214AC -> DP_DEVICES_DIODE
- JP10, JP11, JP12, JP13, JP14, JP15, JP16, JP6, JP7, JP8, JP9: value (none) -> M01; symbol SPARKFUN-CONNECTORS_M01NOSILK-KIT -> SPARKFUN-CONNECTORS_M01
- JP3: value (none) -> SPARKFUN-CONNECTORS_M08; footprint SPARKFUN-CONNECTORS_1X08_NO_SILK -> (none); symbol SPARKFUN-CONNECTORS_M08NO_SILK_FEMALE_PTH -> SPARKFUN-CONNECTORS_M08
- JP5: value (none) -> 1; symbol SPARKFUN-CONNECTORS_M05NO_SILK -> SPARKFUN-CONNECTORS_M05
- R16, R21, R22, R23, R24, R31, R4, R5, R6: symbol ADAFRUIT_R-US_R0603 -> RESISTOR_R-US_
- R28: footprint ADAFRUIT_R0603 -> RESISTOR_R-US_R0603; symbol ADAFRUIT_R-US_R0603 -> RESISTOR_R-US_
- R29: footprint ADAFRUIT_R0603 -> RESISTOR_R0603; symbol ADAFRUIT_R-US_R0603 -> RESISTOR_R-US_
- SJ1: value (none) -> 1; symbol SPARKFUN_SOLDERJUMPER_2WAYS -> SPARKFUN_SOLDERJUMPER_2WAY
- SJ2, SJ3, SJ4, SJ5, SJ6, SJ7: symbol SPARKFUN-RETIRED_SOLDERJUMPERNC -> SPARKFUN-RETIRED_SOLDERJUMPER

Commit message: More Cleaning up
Parts:
- D10, D11, D12, D7, D8, D9: value (none) -> ~
- X14: value USBPTH -> USB; footprint SPARKFUN_USB-B-PTH -> SmoothieBrainz - next round:SPARKFUN_USB-B-PTH
